File: rcbuggtelem/Power.kicad_sch (KiCad schematic)
At the start: 1 part, among them U4 LP38693MP-3.3

Commit message: up
Parts:
- added C10, C11: 1u, Capacitor_SMD:C_0603_1608Metric, symbol Device:C
- added C12, C13: 10u, Capacitor_SMD:C_1210_3225Metric_Pad1.33x2.70mm_HandSolder, symbol Device:C
Connections:
- net VIN: now reaches U4.1 (EN)
- net VIN: now also U4.4 (IN), C10.1, C12.1
- net 3V3: now reaches U4.3 (OUT)
- net 3V3: now also C11.1, C13.1
- net GND: now reaches U4.5 (GND)
- net GND: now also C10.2, C11.2, C12.2, C13.2
