File: rcbuggtelem/MCU.kicad_sch (KiCad schematic)
At the start: 11 parts, among them J4 USB_B_Micro, U1 ESP32-S3-MINI-1

Commit message: update
Parts:
- added J3: Micro_SD_Card, Connector_Card:microSD_HC_Wuerth_693072010801, symbol Connector:Micro_SD_Card
Connections:
- net VUSB renamed Vusb
Changed lines of the file:
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@@
 		)
 	)
-	(global_label "3V3"
+	(hierarchical_label "3V3"
 		(shape input)
 		(at 203.2 41.91 0)
-		(fields_autoplaced yes)
 		(effects
 			(font
@@
 			(justify left)
 		)
-		(property "Intersheetrefs" "${INTERSHEET_REFS}"
-			(at 209.6928 41.91 0)
-			(effects
-				(font
-					(size 1.27 1.27)
-				)
-				(justify left)
-				(hide yes)
-			)
-		)
-	)
-	(global_label "VUSB"
+	)
+	(hierarchical_label "Vusb"
 		(shape input)
 		(at 236.22 81.28 180)
-		(fields_autoplaced yes)
 		(effects
 			(font
@@
 			(justify right)
 		)
-		(property "Intersheetrefs" "${INTERSHEET_REFS}"
-			(at 228.3362 81.28 0)
-			(effects
-				(font
-					(size 1.27 1.27)
-				)
-				(justify right)
-				(hide yes)
-			)
-		)
 	)
 	(symbol
@@
 					(unit 1)
 				)
+			)
+		)
+	)
+	(symbol
+		(lib_id "Connector:Micro_SD_Card")
+		(at 248.92 138.43 0)
+		(unit 1)
+		(exclude_from_sim no)
+		(in_bom yes)
+		(on_board yes)
+		(dnp no)
+		(fields_autoplaced yes)
+		(property "Reference" "J3"
+			(at 249.555 119.38 0)
+			(effects
+				(font
+					(size 1.27 1.27)
+				)
+			)
+		)
+		(property "Value" "Micro_SD_Card"
+			(at 249.555 121.92 0)
+			(effects
+				(font
+					(size 1.27 1.27)
+				)
+			)
+		)
+		(property "Footprint" "Connector_Card:microSD_HC_Wuerth_693072010801"
+			(at 278.13 130.81 0)
+			(effects
+				(font
+					(size 1.27 1.27)
+				)
+				(hide yes)
+			)
+		)
+		(property "Datasheet" "https://www.we-online.com/components/products/datasheet/693072010801.pdf"
+			(at 248.92 138.43 0)
+			(effects
+				(font
+					(size 1.27 1.27)
+				)
+				(hide yes)
+			)
+		)
+		(property "Description" "Micro SD Card Socket"
+			(at 248.92 138.43 0)
+			(effects
+				(font
+					(size 1.27 1.27)
+				)
+				(hide yes)
+			)
+		)
+		(pin "3"
+		)
+		(pin "9"
+		)
+		(pin "4"
+		)
+		(pin "5"
+		)
+		(pin "8"
+		)
+		(pin "7"
+		)
+		(pin "2"
+		)
+		(pin "1"
+		)
+		(pin "6"
+		)
+		(instances
+			(project ""
+				(path "/1aed9cc3-1fd5-4f94-9706-4a914b4693cf/92adddca-c7a8-4d70-9a60-b65170e6c097"
+					(reference "J3")
+					(unit 1)
+				)

Commit message: Signed-off-by: tom <visentin.tom@gmail.com>
Parts:
- added C9: C, symbol Device:C
- added D5: LED, LED_SMD:LED_0603_1608Metric_Pad1.05x0.95mm_HandSolder, symbol Device:LED
- added D6: LED, symbol Device:LED
- added R2, R3, R4, R5, R6: R_US, symbol Device:R_US
Connections:
- net +3.3V: now also J3.4 (VDD), C9.1, R2.1, R3.1, R4.1, R5.2, R6.2
- net GND: now also J3.6 (VSS), J3.9 (SHIELD), C9.2
- net SPI_DO: now reaches U1.15 (IO11)
- net SPI_DO: now also R2.2
- net SPI_DI: now reaches U1.16 (IO12)
- net SPI_DI: now also R3.2
- net SPI_CLK: now reaches U1.17 (IO13)
- net SPI_CLK: now also R4.2
- net CS_ACC: now reaches U1.18 (IO14)
- net CS_MAG: now reaches U1.19 (IO15)
- net ACC_INT: now reaches U1.20 (IO16)
- net MAG_INT: now reaches U1.21 (IO17)
- net at U1.26 (IO26): now also D5.1 (K)
- net at U1.28 (IO33): now also D6.1 (K)
- net at U1.32 (IO36): now also J3.1 (DAT2)
- net at U1.33 (IO37): now also J3.2 (DAT3/CD)
- net at U1.34 (IO38): now also J3.3 (CMD)
- net at U1.35 (IO39): now also J3.5 (CLK)
- net at U1.36 (IO40): now also J3.7 (DAT0)
- net at U1.37 (IO41): now also J3.8 (DAT1)
- new net: D5.2 (A), R5.1
- new net: D6.2 (A), R6.1
Other:
- moved on the sheet: D1, D2, D3, D4, J3, J4

Commit message: up
Parts:
- added C15: 1u, Capacitor_SMD:C_0603_1608Metric, symbol Device:C
- added J5: Conn_01x04_Pin, Connector_PinHeader_2.54mm:PinHeader_1x04_P2.54mm_Vertical, symbol Connector:Conn_01x04_Pin
- added R10, R20, R21, R22, R8, R9: 4k7, Resistor_SMD:R_0603_1608Metric_Pad0.98x0.95mm_HandSolder, symbol Device:R_US
- added SW1: SW_Push, Button_Switch_SMD:SW_SPST_FSMSM, symbol Switch:SW_Push
- C1: value C -> 1u; footprint (none) -> Capacitor_SMD:C_1206_3216Metric
- C2, C3, C4, C9: value C -> 0u1; footprint (none) -> Capacitor_SMD:C_0603_1608Metric
- D1: footprint Diode_THT:D_DO-41_SOD81_P2.54mm_Vertical_AnodeUp -> Diode_SMD:D_SOD-123
- D6: footprint (none) -> LED_SMD:LED_1206_3216Metric
- R1, R2, R3, R4: value R_US -> 4k7; footprint (none) -> Resistor_SMD:R_0603_1608Metric_Pad0.98x0.95mm_HandSolder
- R5, R6: value R_US -> 240R; footprint (none) -> Resistor_SMD:R_0603_1608Metric_Pad0.98x0.95mm_HandSolder
Connections:
- net GND: now also C15.2, R20.1, R21.1, R22.1, SW1.2
- net ADC1: now reaches U1.10 (IO6)
- net ADC2: now reaches U1.11 (IO7)
- net ADC3: now reaches U1.12 (IO8)
- net at U1.27 (IO47): now also J5.4 (Pin_4)
- net at U1.30 (IO48): now also C15.1, SW1.1
- net at U1.38 (IO42): now also J5.1 (Pin_1)
- net at U1.4 (IO0): now also R20.2, R8.2
- net at U1.41 (IO45): now also J5.2 (Pin_2)
- net at U1.44 (IO46): now also J5.3 (Pin_3)
- net at U1.5 (IO1): now also R21.2, R9.2
- net at U1.6 (IO2): now also R10.2, R22.2
- new net CH1_IN: R8.1
- new net CH2_IN: R9.1
- new net CH3_IN: R10.1
Other:
- moved on the sheet: C1, R2, R3, R4

Commit message: up
Parts:
- D5: footprint LED_SMD:LED_0603_1608Metric_Pad1.05x0.95mm_HandSolder -> LED_SMD:LED_1206_3216Metric_Pad1.42x1.75mm_HandSolder
- D6: footprint LED_SMD:LED_1206_3216Metric -> LED_SMD:LED_1206_3216Metric_Pad1.42x1.75mm_HandSolder
Connections:
- net ACC_INT: now also U1.21 (IO17); no longer U1.20 (IO16)
- net CS_ACC: now also U1.19 (IO15); no longer U1.18 (IO14)
- net CS_MAG: now also U1.20 (IO16); no longer U1.19 (IO15)
- net MAG_INT: now also U1.22 (IO18); no longer U1.21 (IO17)
- net SPI_CLK: now also U1.18 (IO14); no longer U1.17 (IO13)
- net SPI_DI: now also U1.17 (IO13); no longer U1.16 (IO12)
- net SPI_DO: now also U1.16 (IO12); no longer U1.15 (IO11)
Other:
- moved on the sheet: R2, R3, R4

Commit message: up
Parts:
- removed C4: 0u1, Capacitor_SMD:C_0603_1608Metric, symbol Device:C
- added R31: DNP, Resistor_SMD:R_0603_1608Metric_Pad0.98x0.95mm_HandSolder, symbol Device:R_US
- C1: footprint Capacitor_SMD:C_1206_3216Metric -> Capacitor_SMD:C_0603_1608Metric_Pad1.08x0.95mm_HandSolder
Connections:
- net ACC_INT: now also U1.15 (IO11); no longer U1.21 (IO17)
- net CS_MAG: now also U1.21 (IO17); no longer U1.20 (IO16)
- net GND: now also J5.4 (Pin_4)
- net at U1.27 (IO47): no longer J5.4 (Pin_4)
- net at U1.39 (TXD0): now also R31.1
- net at U1.40 (RXD0): now also R31.2
Other:
- moved on the sheet: J5, R2, R3, R4
