File: rcbuggtelem/rcbuggtelem.kicad_pcb (KiCad board)
At the start: 2 copper layers, 70 parts, among them J1 Conn_01x10_Pin, J10 SERVO CH 1 OUT, J2 SERVO CH 1 IN, J3 Micro_SD_Card, J4 USB_B_Micro, J5 Conn_01x04_Pin, J6 SERVO CH 1 OUT, J7 SERVO CH 1 IN, J8 SERVO CH 1 OUT, J9 SERVO CH 1 IN, SW1 SW_Push, U1 ESP32-S3-MINI-1, U2 MCP601-xOT, U3 LSM6DSM, U4 LP38693MP-3.3, U5 LIS3MDL, U6 MCP601-xOT, U7 MCP601-xOT

Commit message: up
Parts:
- D5: footprint LED_SMD:LED_0603_1608Metric_Pad1.05x0.95mm_HandSolder -> LED_SMD:LED_1206_3216Metric_Pad1.42x1.75mm_HandSolder
- D6: footprint LED_SMD:LED_1206_3216Metric -> LED_SMD:LED_1206_3216Metric_Pad1.42x1.75mm_HandSolder
- moved SW1 65.9 mm to (77.5, 85.0), turned to 90 degrees
- moved D6 54.2 mm to (82.5, 81.5), turned to 90 degrees
- moved C10 53.0 mm to (50.0, 111.0), turned to 90 degrees
- moved C1 50.3 mm to (123.5, 131.0)
- moved C15 50.3 mm to (96.1, 140.6)
- moved C2 50.3 mm to (96.1, 130.6)
- moved C3 50.3 mm to (96.1, 133.1)
- moved C4 50.3 mm to (96.1, 135.6)
- moved C9 50.3 mm to (96.1, 138.1)
- moved R1 50.3 mm to (95.8, 120.0)
- moved C12 48.1 mm to (49.0, 115.5), turned to -90 degrees
- moved C11 45.5 mm to (59.0, 111.0), turned to 90 degrees
- moved R3 43.9 mm to (86.5, 109.1), turned to 90 degrees
- moved U4 43.6 mm to (54.5, 113.5), turned to 90 degrees
- moved D5 43.3 mm to (82.5, 88.0), turned to 90 degrees
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Connections:
- U1 pad 15: /IMU/SPI_DO -> unconnected-(U1-IO11-Pad15)
- U1 pad 16: /IMU/SPI_DI -> /IMU/SPI_DO
- U1 pad 17: /IMU/SPI_CLK -> /IMU/SPI_DI
- U1 pad 18: /IMU/CS_ACC -> /IMU/SPI_CLK
- U1 pad 19: /IMU/CS_MAG -> /IMU/CS_ACC
- U1 pad 20: /IMU/ACC_INT -> /IMU/CS_MAG
- U1 pad 21: /IMU/MAG_INT -> /IMU/ACC_INT
- U1 pad 22: unconnected-(U1-IO18-Pad22) -> /IMU/MAG_INT
Routing:
- net /MCU/USB_D+: track 0.00 -> 39.6 mm
- net /MCU/USB_D-: track 0.00 -> 38.0 mm
- net /MCU/Vusb: track 0.00 -> 20.9 mm
- net Net-(D1-A): track 0.00 -> 6.18 mm

Commit message: up
Parts:
- added C16: 0u1, Capacitor_SMD:C_0603_1608Metric, F.Cu at (61.8, 111.0)
- added C18: 0u1, Capacitor_SMD:C_0603_1608Metric, F.Cu at (70.2, 105.0)
- added H3: MountingHole, MountingHole:MountingHole_3.2mm_M3, F.Cu at (42.5, 122.8)
- added H4: MountingHole, MountingHole:MountingHole_3.2mm_M3, F.Cu at (83.8, 100.8)
- added R31: DNP, Resistor_SMD:R_0603_1608Metric_Pad0.98x0.95mm_HandSolder, F.Cu at (74.2, 80.2)
- added TP1: TestPoint, TestPoint:TestPoint_Pad_1.0x1.0mm, F.Cu at (63.0, 91.5)
- added TP2: TestPoint, TestPoint:TestPoint_Pad_1.0x1.0mm, F.Cu at (64.0, 93.5)
- added TP3: TestPoint, TestPoint:TestPoint_Pad_1.0x1.0mm, F.Cu at (61.0, 91.5)
- added TP4: TestPoint, TestPoint:TestPoint_Pad_1.0x1.0mm, F.Cu at (55.5, 89.5)
- C1: footprint Capacitor_SMD:C_1206_3216Metric -> Capacitor_SMD:C_0603_1608Metric_Pad1.08x0.95mm_HandSolder
- R2, R3, R4: moved to B.Cu
- moved C3 69.1 mm to (55.8, 77.0), turned to 90 degrees
- moved C2 68.0 mm to (54.2, 77.0), turned to 90 degrees
- moved C1 66.2 mm to (80.8, 80.5), turned to 180 degrees
- moved J1 59.7 mm to (82.2, 121.3), turned to -90 degrees
- moved U2 57.7 mm to (64.5, 113.4), turned to 90 degrees
- moved C14 57.2 mm to (64.5, 116.4), turned to 180 degrees
- moved R24 54.4 mm to (64.5, 110.5), turned to 180 degrees
- moved R23 54.2 mm to (64.5, 109.0)
- moved C6 53.8 mm to (57.0, 100.2)
- moved C9 53.7 mm to (80.5, 86.8), turned to -90 degrees
- moved C15 53.7 mm to (74.5, 91.5), turned to 90 degrees
- moved C5 53.4 mm to (57.0, 98.8)
- moved C8 53.0 mm to (61.5, 98.5), turned to 180 degrees
- moved R7 52.6 mm to (64.5, 118.2)
- moved C7 51.0 mm to (61.5, 100.0), turned to 180 degrees
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Connections:
- J1 pad 1: /PressureSensor/SNS_SUPPLY -> GND
- J1 pad 2: /PressureSensor/SNS_B -> /PressureSensor/SNS_A
- J1 pad 3: /PressureSensor/SNS_A -> /PressureSensor/SNS_B
- J1 pad 4: GND -> /PressureSensor/SNS_SUPPLY
- J10 pad 2: +3V3 -> ServoPower
- J2 pad 2: +3V3 -> ServoPower
- J5 pad 4: Net-(J5-Pin_4) -> GND
- J6 pad 2: +3V3 -> ServoPower
- J7 pad 2: +3V3 -> ServoPower
- J8 pad 2: +3V3 -> ServoPower
- J9 pad 2: +3V3 -> ServoPower
- U1 pad 15: unconnected-(U1-IO11-Pad15) -> /IMU/ACC_INT
- U1 pad 20: /IMU/CS_MAG -> unconnected-(U1-IO16-Pad20)
- U1 pad 21: /IMU/ACC_INT -> /IMU/CS_MAG
- U1 pad 27: Net-(J5-Pin_4) -> unconnected-(U1-IO47-Pad27)
- U1 pad 39: unconnected-(U1-TXD0-Pad39) -> Net-(U1-TXD0)
- U1 pad 40: unconnected-(U1-RXD0-Pad40) -> Net-(U1-RXD0)
Routing:
- net +3V3: track 0.00 -> 48.7 mm, vias 0 -> 20
- net /MCU/ADC1: track 0.00 -> 38.8 mm, vias 0 -> 2
- net /MCU/ADC3: track 0.00 -> 33.3 mm, vias 0 -> 2
- net /MCU/ADC2: track 0.00 -> 31.7 mm, vias 0 -> 2
- net ServoPower: track 0.00 -> 22.9 mm
- net Net-(D6-K): track 0.00 -> 22.8 mm
- net Net-(U1-IO2): track 0.00 -> 21.5 mm
- net Net-(D5-K): track 0.00 -> 20.0 mm
- net Net-(U1-EN): track 0.00 -> 19.3 mm
- net /IMU/SPI_DO: track 0.00 -> 18.5 mm, vias 0 -> 2
- net /IMU/SPI_DI: track 0.00 -> 17.6 mm, vias 0 -> 2
- net /IMU/SPI_CLK: track 0.00 -> 15.2 mm, vias 0 -> 2
- net Net-(U1-IO1): track 0.00 -> 13.3 mm
- net Net-(J5-Pin_1): track 0.00 -> 12.8 mm
- net Net-(J3-DAT0): track 0.00 -> 12.6 mm, vias 0 -> 1
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- added copper zone on In2.Cu, net +3V3
- added copper zone on B.Cu, net GND
- added copper zone on F.Cu, net GND
- added copper zone on In1.Cu, net GND
Other:
- board outline added: 50 x 60.2 mm
- copper layers 2 -> 4
- board text added: "1"
- board text added: "2"
- board text added: "3"
- board text added: "G"
- board text added: "mic"
- board text added: "pwr"
- board text added: "s_sup"
- board text added: "sa"
- board text added: "sb"
- board text added: "temp"
